Commit message: SLAM Workspace

File: my_robot/urdf/beebot1.xacro (robot description, xacro)
@@ -4,5 +4,5 @@
      For more information, please see http://wiki.ros.org/sw_urdf_exporter -->
 <robot name="my_robot1">
-  <link name="robot_footprint">
+  <link name="base_link">
     <inertial>
       <origin
@@ -87,5 +87,5 @@
       rpy="1.5708 0 1.5708" />
     <parent
-      link="robot_footprint" />
+      link="base_link" />
     <child
       link="rmotor" />
@@ -187,5 +187,5 @@
       rpy="-1.5708 0 -1.5708" />
     <parent
-      link="robot_footprint" />
+      link="base_link" />
     <child
       link="lmotor" />
@@ -287,5 +287,5 @@
       rpy="1.5708 0 1.5708" />
     <parent
-      link="robot_footprint" />
+      link="base_link" />
     <child
       link="stud1" />
@@ -337,5 +337,5 @@
       rpy="1.5708 0 1.5708" />
     <parent
-      link="robot_footprint" />
+      link="base_link" />
     <child
       link="stud2" />
@@ -387,5 +387,5 @@
       rpy="1.5708 0 1.5708" />
     <parent
-      link="robot_footprint" />
+      link="base_link" />
     <child
       link="stud3" />
@@ -437,5 +437,5 @@
       rpy="1.5708 0 1.5708" />
     <parent
-      link="robot_footprint" />
+      link="base_link" />
     <child
       link="stud4" />
@@ -488,5 +488,5 @@
       rpy="1.5708 0 1.5708" />
     <parent
-      link="robot_footprint" />
+      link="base_link" />
     <child
       link="front_caster" />
@@ -539,5 +539,5 @@
       rpy="1.5708 0 1.5708" />
     <parent
-      link="robot_footprint" />
+      link="base_link" />
     <child
       link="back_caster" />
@@ -589,5 +589,5 @@
       rpy="1.5708 0 1.5708" />
     <parent
-      link="robot_footprint" />
+      link="base_link" />
     <child
       link="level2" />
@@ -645,5 +645,5 @@
       rpy="1.5708 0 1.5708" />
     <parent
-      link="robot_footprint" />
+      link="base_link" />
     <child
       link="level3" />
@@ -676,5 +676,5 @@
       rpy="0 0 0" />
     <parent
-      link="robot_footprint" />
+      link="base_link" />
     <child link="laser"/>
     <limit effort="1000" lower="0" upper="6.28" velocity="100"/>
@@ -704,5 +704,5 @@
       <odometryTopic>odom</odometryTopic>
       <odometrySource>0</odometrySource>
-      <robotBaseFrame>robot_footprint</robotBaseFrame>
+      <robotBaseFrame>base_link</robotBaseFrame>
       <legacyMode>true</legacyMode>
     </plugin>
